Commit message: rudimentary version of motion execution, squatting motion is (not accurately) tracked by PD

File: src/catkin/motion_planning/momentumopt/src/urdf/quadruped.urdf (robot description, URDF)
Before this commit: robot quadroped, 13 links, 12 joints
Links:
- link BL_contact: geometry collision sphere radius=0.025; visual mesh filename=package://urdf/sphere.obj scale=0.025 0.025 0.025
- link BL_shank: geometry collision cylinder length=0.16 radius=0.025; visual mesh filename=package://urdf/cylinder.obj scale=0.025 0.025 0.16
- link BL_upperleg: geometry collision cylinder length=0.16 radius=0.025; visual mesh filename=package://urdf/cylinder.obj scale=0.025 0.025 0.16
- link BR_contact: geometry collision sphere radius=0.025; visual mesh filename=package://urdf/sphere.obj scale=0.025 0.025 0.025
- link BR_shank: geometry collision cylinder length=0.16 radius=0.025; visual mesh filename=package://urdf/cylinder.obj scale=0.025 0.025 0.16
- link BR_upperleg: geometry collision cylinder length=0.16 radius=0.025; visual mesh filename=package://urdf/cylinder.obj scale=0.025 0.025 0.16
- link FL_contact: geometry collision sphere radius=0.025; visual mesh filename=package://urdf/sphere.obj scale=0.025 0.025 0.025
- link FL_shank: geometry collision cylinder length=0.16 radius=0.025; visual mesh filename=package://urdf/cylinder.obj scale=0.025 0.025 0.16
- link FL_upperleg: geometry collision cylinder length=0.16 radius=0.025; visual mesh filename=package://urdf/cylinder.obj scale=0.025 0.025 0.16
- link FR_contact: geometry collision sphere radius=0.025; visual mesh filename=package://urdf/sphere.obj scale=0.025 0.025 0.025
- link FR_shank: geometry collision cylinder length=0.16 radius=0.025; visual mesh filename=package://urdf/cylinder.obj scale=0.025 0.025 0.16
- link FR_upperleg: geometry collision cylinder length=0.16 radius=0.025; visual mesh filename=package://urdf/cylinder.obj scale=0.025 0.025 0.16
- link base_link: geometry collision box size=0.2 0.4 0.05; visual mesh filename=package://urdf/cube.obj scale=0.2 0.4 0.05

Commit message: Remove the old quadruped URDF files

File: src/catkin/motion_planning/momentumopt/src/urdf/quadruped.urdf (robot description, URDF)
Before this commit: robot quadroped, 13 links, 12 joints
Links:
- removed link BL_contact
- removed link BL_shank
- removed link BL_upperleg
- removed link BR_contact
- removed link BR_shank
- removed link BR_upperleg
- removed link FL_contact
- removed link FL_shank
- removed link FL_upperleg
- removed link FR_contact
- removed link FR_shank
- removed link FR_upperleg
- added link FL_FOOT, mass 0.01; collision mesh filename=package://urdf/obj/with_foot/quadruped_foot.obj; visual mesh filename=package://urdf/obj/with_foot/quadruped_foot.obj
- added link FL_LOWER_LEG, mass 0.021; collision mesh filename=package://urdf/obj/with_foot/quadruped_lower_leg_left_side.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; visual mesh filename=package://urdf/obj/with_foot/quadruped_lower_leg_left_side.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
- added link FL_UPPER_LEG, mass 0.162; collision mesh filename=package://urdf/obj/with_foot/quadruped_upper_leg_left_side.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; visual mesh filename=package://urdf/obj/with_foot/quadruped_upper_leg_left_side.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
- added link FR_FOOT, mass 0.01; collision mesh filename=package://urdf/obj/with_foot/quadruped_foot.obj; visual mesh filename=package://urdf/obj/with_foot/quadruped_foot.obj
- added link FR_LOWER_LEG, mass 0.021; collision mesh filename=package://urdf/obj/with_foot/quadruped_lower_leg_right_side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; visual mesh filename=package://urdf/obj/with_foot/quadruped_lower_leg_right_side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
- added link FR_UPPER_LEG, mass 0.162; collision mesh filename=package://urdf/obj/with_foot/quadruped_upper_leg_right_side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; visual mesh filename=package://urdf/obj/with_foot/quadruped_upper_leg_right_side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
- added link HL_FOOT, mass 0.01; collision mesh filename=package://urdf/obj/with_foot/quadruped_foot.obj; visual mesh filename=package://urdf/obj/with_foot/quadruped_foot.obj
- added link HL_LOWER_LEG, mass 0.021; collision mesh filename=package://urdf/obj/with_foot/quadruped_lower_leg_left_side.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; visual mesh filename=package://urdf/obj/with_foot/quadruped_lower_leg_left_side.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
- added link HL_UPPER_LEG, mass 0.162; collision mesh filename=package://urdf/obj/with_foot/quadruped_upper_leg_left_side.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; visual mesh filename=package://urdf/obj/with_foot/quadruped_upper_leg_left_side.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
- added link HR_FOOT, mass 0.01; collision mesh filename=package://urdf/obj/with_foot/quadruped_foot.obj; visual mesh filename=package://urdf/obj/with_foot/quadruped_foot.obj
- added link HR_LOWER_LEG, mass 0.021; collision mesh filename=package://urdf/obj/with_foot/quadruped_lower_leg_right_side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; visual mesh filename=package://urdf/obj/with_foot/quadruped_lower_leg_right_side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
- added link HR_UPPER_LEG, mass 0.162; collision mesh filename=package://urdf/obj/with_foot/quadruped_upper_leg_right_side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; visual mesh filename=package://urdf/obj/with_foot/quadruped_upper_leg_right_side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
- link base_link: geometry collision mesh filename=package://urdf/obj/with_foot/quadruped_body.obj; visual mesh filename=package://urdf/obj/with_foot/quadruped_body.obj
Joints:
- removed joint BL_END
- removed joint BL_HFE
- removed joint BL_KFE
- removed joint BR_END
- removed joint BR_HFE
- removed joint BR_KFE
- removed joint FL_END
- removed joint FR_END
- added joint FL_ANKLE: type fixed, parent FL_LOWER_LEG, child FL_FOOT, origin xyz=0 0 -0.16 rpy=0 0 0, limit lower=-10 upper=10 effort=1000 velocity=1000
- added joint FR_ANKLE: type fixed, parent FR_LOWER_LEG, child FR_FOOT, origin xyz=0 0 -0.16 rpy=0 0 0, limit lower=-10 upper=10 effort=1000 velocity=1000
- added joint HL_ANKLE: type fixed, parent HL_LOWER_LEG, child HL_FOOT, origin xyz=0 0 -0.16 rpy=0 0 0, limit lower=-10 upper=10 effort=1000 velocity=1000
- added joint HL_HFE: type revolute, parent base_link, child HL_UPPER_LEG, origin xyz=-0.19 0.1046 0 rpy=0 0 0, axis 0 1 0, limit lower=-10 upper=10 effort=1000 velocity=1000
- added joint HL_KFE: type revolute, parent HL_UPPER_LEG, child HL_LOWER_LEG, origin xyz=0 0.03745 -0.16 rpy=0 0 0, axis 0 1 0, limit lower=-10 upper=10 effort=1000 velocity=1000
- added joint HR_ANKLE: type fixed, parent HR_LOWER_LEG, child HR_FOOT, origin xyz=0 0 -0.16 rpy=0 0 0, limit lower=-10 upper=10 effort=1000 velocity=1000
- added joint HR_HFE: type revolute, parent base_link, child HR_UPPER_LEG, origin xyz=-0.19 -0.1046 0 rpy=0 0 0, axis 0 1 0, limit lower=-10 upper=10 effort=1000 velocity=1000
- added joint HR_KFE: type revolute, parent HR_UPPER_LEG, child HR_LOWER_LEG, origin xyz=0 -0.03745 -0.16 rpy=0 0 0, axis 0 1 0, limit lower=-10 upper=10 effort=1000 velocity=1000
- joint FL_HFE: axis 1 0 0 -> 0 1 0; child FL_upperleg -> FL_UPPER_LEG; origin xyz=-0.1 0.2 0 rpy=0 0 0 -> xyz=0.19 0.1046 0 rpy=0 0 0
- joint FL_KFE: axis 1 0 0 -> 0 1 0; child FL_shank -> FL_LOWER_LEG; limit effort=1000 velocity=10000 -> lower=-10 upper=10 effort=1000 velocity=1000; origin xyz=0 0 -0.16 rpy=0 0 0 -> xyz=0 0.03745 -0.16 rpy=0 0 0; parent FL_upperleg -> FL_UPPER_LEG
- joint FR_HFE: axis 1 0 0 -> 0 1 0; child FR_upperleg -> FR_UPPER_LEG; origin xyz=0.1 0.2 0 rpy=0 0 0 -> xyz=0.19 -0.1046 0 rpy=0 0 0
- joint FR_KFE: axis 1 0 0 -> 0 1 0; child FR_shank -> FR_LOWER_LEG; limit effort=1000 velocity=10000 -> lower=-10 upper=10 effort=1000 velocity=1000; origin xyz=0 0 -0.16 rpy=0 0 0 -> xyz=0 -0.03745 -0.16 rpy=0 0 0; parent FR_upperleg -> FR_UPPER_LEG
